File: EMFDetector-PCB/Version_2/EMFDetector_v2.sch (KiCad schematic (older format))
At the start: 25 parts, among them J1 PHONO, P1 BATT, P2 BATT, P3 PCB, P4 LOGO1, P5 LOGO2, SW1 PWR, U1 OPA2134

Commit message: New version of PCB built for new kicad version
Parts:
- L1, L2: symbol pspice:INDUCTOR -> Device:L
- P4: footprint CuriousElectric3:CuriousElectric_flat_12mm -> CuriousElectric3:TCEC_Words_13mm
Connections:
- net GND: now also J1.1 (S); no longer J1.2 (T)
- net at C6.1: now also J1.2 (T); no longer J1.1 (S)
Changed lines of the file:
@@
 $EndComp
 $Comp
-L pspice:INDUCTOR L1
+L Device:L L1
 U 1 1 574B4587
 P 5350 2850
@@
 F 3 "" H 5350 2850 50  0000 C CNN
 	1    5350 2850
-	0    1    1    0
-$EndComp
-$Comp
-L pspice:INDUCTOR L2
+	1    0    0    -1
+$EndComp
+$Comp
+L Device:L L2
 U 1 1 574B46BA
 P 5350 4450
@@
 F 3 "" H 5350 4450 50  0000 C CNN
 	1    5350 4450
-	0    1    1    0
+	1    0    0    -1
 $EndComp
 $Comp
@@
 L matts_components:GND #PWR011
 U 1 1 574B62D1
-P 7950 2950
-F 0 "#PWR011" H 7950 2700 50  0001 C CNN
-F 1 "GND" H 7950 2800 50  0000 C CNN
-F 2 "" H 7950 2950 50  0000 C CNN
-F 3 "" H 7950 2950 50  0000 C CNN
-	1    7950 2950
-	1    0    0    -1
-$EndComp
-Wire Wire Line
-	7950 2950 7950 2850
-Wire Wire Line
-	7950 2850 9350 2850
+P 9250 3150
+F 0 "#PWR011" H 9250 2900 50  0001 C CNN
+F 1 "GND" H 9250 3000 50  0000 C CNN
+F 2 "" H 9250 3150 50  0000 C CNN
+F 3 "" H 9250 3150 50  0000 C CNN
+	1    9250 3150
+	1    0    0    -1
+$EndComp
+Wire Wire Line
+	9250 3150 9250 3050
 $Comp
 L power:VCC #PWR09
@@
 	2400 2750 3700 2750
 Wire Wire Line
-	7950 4150 9200 4150
+	7950 4150 9050 4150
 Wire Wire Line
 	9200 2650 9350 2650
@@
 F 0 "P4" H 9550 4200 50  0000 C CNN
 F 1 "LOGO1" V 9650 4100 50  0000 C CNN
-F 2 "CuriousElectric3:CuriousElectric_flat_12mm" H 9550 4100 50  0001 C CNN
+F 2 "CuriousElectric3:TCEC_Words_13mm" H 9550 4100 50  0001 C CNN
 F 3 "" H 9550 4100 50  0000 C CNN
 	1    9550 4100
@@
 	1    0    0    -1
 $EndComp
-Wire Wire Line
-	9200 4150 9200 3050
-Wire Wire Line
-	9200 3050 9350 3050
 $Comp
 L Device:LED D1
@@
 	4650 2000 4650 2200
 Wire Wire Line
-	5350 2500 5350 2600
-Wire Wire Line
-	5350 3100 5350 3600
-Wire Wire Line
-	5350 3600 5350 4200
-Wire Wire Line
-	5350 4700 5350 4800
+	5350 3600 5350 4300
+Wire Wire Line
+	5350 4600 5350 4800
+Wire Wire Line
+	5350 3000 5350 3600
+Wire Wire Line
+	5350 2500 5350 2700
+Wire Wire Line
+	9350 3050 9250 3050
+Wire Wire Line
+	9350 2850 9050 2850
+Wire Wire Line
+	9050 2850 9050 4150
 $EndSCHEMATC
